Commit message: Offsets work and moveit works IRL! :)

File: zebmite_ws/src/minifrcrobot_description/urdf/robot.urdf (robot description, URDF)
Before this commit: robot onshape, 4 links, 3 joints
Joints:
- joint base_arm: limit lower=-1.7 upper=1.5 effort=10000 velocity=20 -> lower=-0.296706 upper=1.274 effort=10000 velocity=200000
- joint second_stage_arm: limit lower=-2.0 upper=4.5 effort=1000000 velocity=20 -> lower=-1.13446 upper=0.43633 effort=1000000 velocity=200000

Commit message: MOVEIT IS CRAZY

File: zebmite_ws/src/minifrcrobot_description/urdf/robot.urdf (robot description, URDF)
Before this commit: robot onshape, 4 links, 3 joints
Joints:
- joint base_arm: limit lower=-0.296706 upper=1.274 effort=10000 velocity=200000 -> lower=-2.14 upper=5.14 effort=10000 velocity=200000
- joint second_stage_arm: limit lower=-1.13446 upper=0.43633 effort=1000000 velocity=200000 -> lower=-3.14 upper=3.14 effort=1000000 velocity=200000

Commit message: new urdf

File: zebmite_ws/src/minifrcrobot_description/urdf/robot.urdf (robot description, URDF)
Before this commit: robot onshape, 4 links, 3 joints
Links:
- removed link sg90-micro-servo-9g-tower-pro-1.snapshot.3
- removed link sg90_-_micro_servo_9g_-_tower_pro.3
- added link _hs-322hd, mass 0.049980665650601885375; collision mesh filename=package:///_hs-322hd_collision.stl; visual box size=0 0 0
- added link _hs-322hd_1, mass 1e-9; visual mesh filename=package:///_hs-322hd.stl
- added link arm_holder, mass 0.038331078295993678551; collision mesh filename=package:///arm_holder_collision.stl; visual box size=0 0 0
- added link arm_holder_1, mass 1e-9; visual mesh filename=package:///arm_holder.stl
- added link base_arm_part, mass 0.035980036837035184183; collision mesh filename=package:///base_arm_part_collision.stl; visual box size=0 0 0
- added link base_arm_part_1, mass 1e-9; visual mesh filename=package:///base_arm_part.stl
- added link part_1_1, mass 1e-9; visual mesh filename=package:///part_1.stl
- link part_1: mass 0.01868093335900054483 -> 0.023127123465820405984; geometry collision mesh filename=package:///part_1_collision.stl; visual box size=0 0 0
Joints:
- added joint _hs-322hd_1_fixing: type fixed, parent _hs-322hd, child _hs-322hd_1, origin xyz=0 0 0 rpy=0 -0 0, axis 0 0 1, limit effort=1 velocity=20
- added joint arm_holder_1_fixing: type fixed, parent arm_holder, child arm_holder_1, origin xyz=0 0 0 rpy=0 -0 0, axis 0 0 1, limit effort=1 velocity=20
- added joint base_arm_part_1_fixing: type fixed, parent base_arm_part, child base_arm_part_1, origin xyz=0 0 0 rpy=0 -0 0, axis 0 0 1, limit effort=1 velocity=20
- added joint part_1_1_fixing: type fixed, parent part_1, child part_1_1, origin xyz=0 0 0 rpy=0 -0 0, axis 0 0 1, limit effort=1 velocity=20
- added joint servo_link: type fixed, parent arm_holder, child _hs-322hd, origin xyz=0.022224999999999998229 -6.9388939039072283776e-18 0.025400000000000016315 rpy=-1.570796326794896558 1.5707963267948961139 0, axis 0 0 1, limit effort=1 velocity=20
- joint base_arm: child part_1 -> base_arm_part; limit lower=-2.14 upper=5.14 effort=10000 velocity=200000 -> effort=1 velocity=20; origin xyz=0.0056499999999999848954 3.0357660829594124152e-16 0.03350000000000099426 rpy=1.570796326794896336 -0.15085086535037292577 1.570796326794896558 -> xyz=-0.010000000000000997674 0.011600000000000769418 -1.6316198063596397266e-09 rpy=-1.5707963793909751615 1.5686835501809441862 3.1415926009938330843; parent sg90_-_micro_servo_9g_-_tower_pro.3 -> _hs-322hd
- joint base_link_to_base: child sg90_-_micro_servo_9g_-_tower_pro.3 -> arm_holder
- joint second_stage_arm: child sg90-micro-servo-9g-tower-pro-1.snapshot.3 -> part_1; limit lower=-3.14 upper=3.14 effort=1000000 velocity=200000 -> effort=1 velocity=20; origin xyz=-8.6736173798840354721e-19 0.22804154362529510669 8.6736173798840354721e-19 rpy=-3.141592653589793116 8.0835220919448662387e-22 2.6097509957447053708 -> xyz=-1.4297916149652589723e-17 -0.26589736000000013805 -0.030797499999999207454 rpy=1.1408386409076440936e-16 8.8940818644187655745e-17 0.0016804094650094574849; parent part_1 -> base_arm_part

Commit message: latest urdf

File: zebmite_ws/src/minifrcrobot_description/urdf/robot.urdf (robot description, URDF)
Before this commit: robot onshape, 9 links, 8 joints
Links:
- link _hs-322hd: geometry collision mesh filename=package://minifrcrobot_description/urdf/_hs-322hd_collision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; visual box size=0 0 0
- link _hs-322hd_1: geometry visual mesh filename=package://minifrcrobot_description/urdf/_hs-322hd.stl
- link arm_holder: mass 0.038331078295993678551 -> 0.040789137895993712868; geometry collision mesh filename=package://minifrcrobot_description/urdf/arm_holder_collisio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; visual box size=0 0 0
- link arm_holder_1: geometry visual mesh filename=package://minifrcrobot_description/urdf/arm_holder.stl
- link base_arm_part: mass 0.035980036837035184183 -> 0.035980036837035156427; geometry collision mesh filename=package://minifrcrobot_description/urdf/base_arm_part_colli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; visual box size=0 0 0
- link base_arm_part_1: geometry visual mesh filename=package://minifrcrobot_description/urdf/base_arm_part.stl
- link part_1: geometry collision mesh filename=package://minifrcrobot_description/urdf/part_1_collision.stl; visual box size=0 0 0
- link part_1_1: geometry visual mesh filename=package://minifrcrobot_description/urdf/part_1.stl
Joints:
- joint base_arm: limit effort=1 velocity=20 -> lower=-6.28 upper=6.28 effort=1 velocity=20; origin xyz=-0.010000000000000997674 0.011600000000000769418 -1.6316198063596397266e-09 rpy=-1.5707963793909751615 1.5686835501809441862 3.1415926009938330843 -> xyz=-0.010000000000000997674 0.011599999999999995731 -1.6316197924818519188e-09 rpy=-1.5707963793909751615 1.5686835501809441862 3.1415926009938330843
- joint second_stage_arm: limit effort=1 velocity=20 -> lower=-6.28 upper=6.28 effort=1 velocity=20; origin xyz=-1.4297916149652589723e-17 -0.26589736000000013805 -0.030797499999999207454 rpy=1.1408386409076440936e-16 8.8940818644187655745e-17 0.0016804094650094574849 -> xyz=4.336808689942017736e-19 -0.26589736000000008254 -0.028257499999999977081 rpy=1.1408386409076440936e-16 8.8940818644187655745e-17 0.0016804094650094574849
- joint servo_link: origin xyz=0.022224999999999998229 -6.9388939039072283776e-18 0.025400000000000016315 rpy=-1.570796326794896558 1.5707963267948961139 0 -> xyz=0.028574999999999999706 -6.9388939039072283776e-18 0.025400000000000016315 rpy=-1.570796326794896558 1.5707963267948961139 0

Commit message: make urdf stop complaining

File: zebmite_ws/src/minifrcrobot_description/urdf/robot.urdf (robot description, URDF)
Before this commit: robot onshape, 9 links, 8 joints
Links:
- added link bl_drive_link
- added link br_drive_link
- added link fl_drive_link
- added link fr_drive_link
- added link intake_link
Joints:
- added joint bl_drive: type fixed, parent base_link, child bl_drive_link, origin xyz=0 0 0 rpy=0.0 0 0
- added joint br_drive: type fixed, parent base_link, child br_drive_link, origin xyz=0 0 0 rpy=0.0 0 0
- added joint fl_drive: type fixed, parent base_link, child fl_drive_link, origin xyz=0 0 0 rpy=0.0 0 0
- added joint fr_drive: type fixed, parent base_link, child fr_drive_link, origin xyz=0 0 0 rpy=0.0 0 0
- added joint intake: type fixed, parent base_link, child intake_link, origin xyz=0 0 0 rpy=0.0 0 0

Commit message: p

File: zebmite_ws/src/minifrcrobot_description/urdf/robot.urdf (robot description, URDF)
Before this commit: robot onshape, 14 links, 13 joints
Joints:
- joint base_arm: limit lower=-6.28 upper=6.28 effort=1 velocity=20 -> lower=-1.6 upper=1.6 effort=1 velocity=20

Commit message: start adding arm positions

File: zebmite_ws/src/minifrcrobot_description/urdf/robot.urdf (robot description, URDF)
Before this commit: robot onshape, 14 links, 13 joints
Joints:
- joint base_arm: limit lower=-1.6 upper=1.6 effort=1 velocity=20 -> lower=-1.22 upper=1.6 effort=1 velocity=0.1
- joint second_stage_arm: limit lower=-6.28 upper=6.28 effort=1 velocity=20 -> lower=-2.2 upper=1.6 effort=1 velocity=0.1

Commit message: add more positions

File: zebmite_ws/src/minifrcrobot_description/urdf/robot.urdf (robot description, URDF)
Before this commit: robot onshape, 14 links, 13 joints
Joints:
- joint base_arm: limit lower=-1.22 upper=1.6 effort=1 velocity=0.1 -> lower=-1.22 upper=1.6 effort=1 velocity=5.0
- joint second_stage_arm: limit lower=-2.2 upper=1.6 effort=1 velocity=0.1 -> lower=-2.2 upper=1.6 effort=1 velocity=5.0

Commit message: auto

File: zebmite_ws/src/minifrcrobot_description/urdf/robot.urdf (robot description, URDF)
Before this commit: robot onshape, 14 links, 13 joints
Links:
- added link auto_motor_link
Joints:
- added joint auto_motor: type fixed, parent base_link, child auto_motor_link, origin xyz=0 0 0 rpy=0.0 0 0

Commit message: backup from chris's computer

File: zebmite_ws/src/minifrcrobot_description/urdf/robot.urdf (robot description, URDF)
Before this commit: robot onshape, 15 links, 14 joints
Joints:
- joint base_arm: limit lower=-1.22 upper=1.6 effort=1 velocity=5.0 -> lower=-1.22 upper=1.6 effort=1 velocity=3.14

Commit message: websockets works

File: zebmite_ws/src/minifrcrobot_description/urdf/robot.urdf (robot description, URDF)
Before this commit: robot onshape, 15 links, 14 joints
Links:
- removed link auto_motor_link
- added link test_servo_link
Joints:
- removed joint auto_motor
- added joint test_servo: type fixed, parent base_link, child test_servo_link, origin xyz=0 0 0 rpy=0.0 0 0

Commit message: changes

File: zebmite_ws/src/minifrcrobot_description/urdf/robot.urdf (robot description, URDF)
Before this commit: robot onshape, 15 links, 14 joints
Links:
- added link top_intake_link
Joints:
- added joint intake_top_roller: type revolute, parent base_link, child top_intake_link, origin xyz=0 0 0 rpy=0.0 0 0, limit effort=1 velocity=20
- joint bl_drive: axis (none) -> 0 0 1; limit (none) -> effort=1 velocity=20; origin xyz=0 0 0 rpy=0.0 0 0 -> xyz=69 1 1 rpy=0.0 0 0; type fixed -> revolute
- joint br_drive: limit (none) -> effort=1 velocity=20; type fixed -> revolute
- joint fl_drive: limit (none) -> effort=1 velocity=20; type fixed -> revolute
- joint fr_drive: limit (none) -> effort=1 velocity=20; type fixed -> revolute
- joint intake: limit (none) -> effort=1 velocity=20; type fixed -> revolute
- joint test_servo: limit (none) -> effort=1 velocity=20; type fixed -> revolute
